Commit message: Modify the panda urdf for the additional frame

File: tf_robot_learning/data/urdf/panda_arm.urdf (robot description, URDF)
Before this commit: robot panda, 11 links, 10 joints
Links:
- added link panda_hand2
Joints:
- added joint panda_hand_joint2: type fixed, parent panda_hand, child panda_hand2, origin xyz=0 0 0 rpy=0  0

File: tf_robot_learning/data/urdf/panda_arm_gripper.urdf (robot description, URDF)
Before this commit: robot panda, 14 links, 13 joints
Links:
- added link panda_hand2
Joints:
- added joint panda_hand_joint2: type fixed, parent panda_hand, child panda_hand2, origin xyz=0 0 0 rpy=0  0
