Commit message: At submission of revised paper

File: tf_robot_learning/data/urdf/bookshelf_simple_collision.urdf (robot description, URDF)
Before this commit: robot bookcase, 4 links, 3 joints
Links:
- link bookcase: geometry collision box size=0.02 0.4 1.4; collision box size=0.02 0.4 1.4

Commit message: Before removing old codes

File: tf_robot_learning/data/urdf/bookshelf_simple_collision.urdf (robot description, URDF)
Before this commit: robot bookcase, 4 links, 3 joints
Links:
- link bookcase: geometry collision box size=0.02 0.4 1.4; collision box size=0.02 0.4 1.4

File: tf_robot_learning/data/urdf/panda_arm.urdf (robot description, URDF)
Before this commit: robot panda, 12 links, 11 joints
Links:
- link panda_hand2: geometry visual box size=0.0001 0.0001 0.0001
Joints:
- joint panda_hand_joint2: origin xyz=0 0 0 rpy=0  0 -> xyz=0 0 0 rpy=0 -1.5707963 0
