Commit message: Setting up the walker rrt

File: tf_robot_learning/data/urdf/walker_description/urdf/walker_simple.urdf (robot description, URDF)
Before this commit: robot walker, 63 links, 62 joints
Joints:
- joint head_j1: type revolute -> fixed
- joint head_j2: type revolute -> fixed
- joint left_index_j1: type revolute -> fixed
- joint left_index_j2: type revolute -> fixed
- joint left_middle_j1: type revolute -> fixed
- joint left_middle_j2: type revolute -> fixed
- joint left_pinky_j1: type revolute -> fixed
- joint left_pinky_j2: type revolute -> fixed
- joint left_ring_j1: type revolute -> fixed
- joint left_ring_j2: type revolute -> fixed
- joint left_thumb_j1: type revolute -> fixed
- joint left_thumb_j2: type revolute -> fixed
- joint right_index_j1: type revolute -> fixed
- joint right_index_j2: type revolute -> fixed
- joint right_middle_j1: type revolute -> fixed
- joint right_middle_j2: type revolute -> fixed
- joint right_pinky_j1: type revolute -> fixed
- joint right_pinky_j2: type revolute -> fixed
- joint right_ring_j1: type revolute -> fixed
- joint right_ring_j2: type revolute -> fixed
- joint right_thumb_j1: type revolute -> fixed
- joint right_thumb_j2: type revolute -> fixed
